File: Smart Key Cutter Interface.kicad_pcb (KiCad board)
At the start: 4 copper layers, 80 x 96 mm, 114 parts, among them J1 Battery, J10 LED-SWITCH, J2 Encoder, J3 Encoder, J4 124018612112A, J5 503398-1892, J6 M5-Power, J7 M5-RED, J8 Conn_01x03, J9 Feeltech, M1 NEMA8, M2 NEMA8, Q1 L8050QLT1G, Q2 L8050QLT1G, Q3 G230P06K, SW1 SW_Push, SW2 SW_Push, SW3 ON/OFF, U1 TXU0104PWR, U10 AM26C32IDR, U12 AM26C32IDR, U13 USBLC6-2SC6, U14 3S Charger, U15 MAX3485, U2 TXU0104PWR, U3 SN74HC4066PWR, U4 CP2102N-Axx-xQFN28, U5 ESP32-S3-WROOM-1-N16, U6 INA228, U7 AMS1117-3.3, U8 TPS82130

Commit message: Version 2 sent to JLC
Parts:
- removed C13: 100nF, Capacitor_SMD:C_0402_1005Metric
- removed C40: 68uF, Capacitor_SMD:C_2220_5750Metric
- added TP1: TestPoint, Ingenium:RH-5015, F.Cu at (91.8, 49.5)
- D1: value SK6812 -> LED; footprint LED_SMD:LED_SK6812_PLCC4_5.0x5.0mm_P3.2mm -> LED_SMD:LED_0603_1608Metric
- R13: value 0 -> 280
- R14, R15: value 10k -> 22k
- moved J10 101.8 mm to (81.4, 51.7), turned to -90 degrees
- moved R32 100.7 mm to (84.7, 50.0), turned to -90 degrees
- moved J7 99.0 mm to (145.3, 132.3), turned to 90 degrees
- moved J3 97.4 mm to (72.2, 64.5), turned to -90 degrees
- moved C14 94.3 mm to (150.5, 72.1), turned to -90 degrees
- moved C3 87.9 mm to (146.9, 122.0), turned to 0 degrees
- moved J1 87.1 mm to (142.5, 67.9), turned to 90 degrees
- moved C36 86.7 mm to (85.6, 58.5), turned to 180 degrees
- moved U6 86.5 mm to (147.5, 74.7), turned to 90 degrees
- moved J8 85.9 mm to (149.0, 117.1), turned to 90 degrees
- moved J2 80.0 mm to (72.3, 78.3), turned to -90 degrees
- moved U12 79.7 mm to (84.1, 64.5), turned to 0 degrees
- moved R16 79.4 mm to (143.5, 75.1), turned to -90 degrees
- moved J6 78.1 mm to (81.4, 129.1)
- moved C1 77.5 mm to (141.6, 121.7), turned to 0 degrees
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Connections:
- net /Connectors/RS485_DI renamed /RS485_DI
- net /Connectors/RS485_DIR renamed /RS485_DIR
- net /Connectors/RS485_RO renamed /RS485_RO
- net /MCU/GPIO48 renamed Net-(U5-IO48)
- J8 pad 1: +5V -> GND
- J8 pad 3: GND -> +5V
- R14 pad 1: Net-(U6-A1) -> +3V3
- R14 pad 2: GND -> /Motor_UART_1
- R15 pad 1: Net-(U6-A0) -> +3V3
- R15 pad 2: GND -> /Motor_UART_2
- U6 pad 1: Net-(U6-A1) -> GND
- U6 pad 2: Net-(U6-A0) -> GND
- U6 pad 4: /I2C_SCL -> /I2C_SDA
- U6 pad 5: /I2C_SDA -> /I2C_SCL
Routing:
- net /LED_SWITCH: track 51.7 -> 130.6 mm, vias 2 -> 1
- net /I2C_SDA: track 134.3 -> 83.1 mm
- net /Motor_Enable_2: track 84.3 -> 38.9 mm
- net /SCK: track 139.1 -> 102.9 mm
- net /SD_CS: track 145.9 -> 109.7 mm
- net /Motor_Enable_1: track 61.2 -> 25.9 mm, vias 2 -> 4
- net /MISO: track 138.9 -> 106.7 mm, vias 2 -> 4
- net +5V: track 189.0 -> 215.9 mm
- net /LED_DATA_3V3: track 64.5 -> 39.3 mm, vias 2 -> 0
- net /Motor_Stall_2: track 60.1 -> 39.0 mm, vias 4 -> 2
- net /Motor_Stall_1: track 49.3 -> 28.3 mm
- net /Motor_STEP_1: track 45.7 -> 25.4 mm
- net /CH_A_5V_1: track 34.6 -> 53.9 mm
- net /I2C_SCL: track 111.2 -> 93.7 mm, vias 3 -> 1
- net /Motor_UART_1: track 29.0 -> 45.8 mm, vias 0 -> 2
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- added copper zone on F.Cu, net +3V3
Other:
- board text added: "{ "ViaStitching": "0.2", "stitch_zone_0": { "HSpacing": "1", "VSpacing": "1", "HOffset": "0", "VOffset": "0", "Clearance": "0", "Randomize": true } }"
